File: esp8266/esp8266.sch (KiCad schematic (older format))
At the start: 18 parts, among them J1 Screw_Terminal_1x02, J2 Screw_Terminal_1x03, P1 CONN_02X04, P2 CONN_01X03, P3 CONN_01X03, P4 CONN_01X03, P5 CONN_01X03, P6 CONN_01X03, U1 LM1117-3.3

Commit message: changed to LD1117
Parts:
- removed U1: LM1117-3.3, TO_SOT_Packages_THT:TO-220_Neutral123_Vertical, symbol LM1117-3.3
- added U1: LD1117S33TR, TO_SOT_Packages_THT:TO-220_Neutral123_Vertical, symbol LD1117S33TR
Changed lines of the file:
@@
 U 1 1 5823A171
 P 5300 3150
-F 0 "P1" H 5300 3400 50  0000 C CNN
-F 1 "CONN_02X04" H 5300 2900 50  0000 C CNN
+F 0 "P1" H 5300 3515 50  0000 C CNN
+F 1 "CONN_02X04" H 5300 3424 50  0000 C CNN
 F 2 "Socket_Strips:Socket_Strip_Straight_2x04" H 5300 1950 50  0001 C CNN
 F 3 "" H 5300 1950 50  0000 C CNN
 	1    5300 3150
 	-1   0    0    -1
-$EndComp
-$Comp
-L LM1117-3.3 U1
-U 1 1 5823A275
-P 6050 1600
-F 0 "U1" H 6150 1350 50  0000 C CNN
-F 1 "LM1117-3.3" H 6050 1850 50  0000 C CNN
-F 2 "TO_SOT_Packages_THT:TO-220_Neutral123_Vertical" H 6050 1600 50  0001 C CNN
-F 3 "" H 6050 1600 50  0000 C CNN
-	1    6050 1600
-	1    0    0    -1
 $EndComp
 $Comp
@@
 $EndComp
 Wire Wire Line
-	6350 1600 6900 1600
+	6450 1600 6900 1600
 Connection ~ 6750 1600
 Wire Wire Line
-	4800 1600 5750 1600
+	4800 1600 5650 1600
 Connection ~ 4950 1600
 Wire Wire Line
@@
 U 1 1 5824B234
 P 1500 2750
-F 0 "P3" V 1465 2928 50  0000 L CNN
-F 1 "CONN_01X03" V 1374 2928 50  0000 L CNN
+F 0 "P3" V 1715 2745 50  0000 C CNN
+F 1 "CONN_01X03" V 1624 2745 50  0000 C CNN
 F 2 "Socket_Strips:Socket_Strip_Straight_1x03" H 1500 2750 50  0001 C CNN
 F 3 "" H 1500 2750 50  0000 C CNN
@@
 U 1 1 5824B805
 P 2300 2750
-F 0 "P5" V 2265 2928 50  0000 L CNN
-F 1 "CONN_01X03" V 2174 2928 50  0000 L CNN
+F 0 "P5" V 2515 2745 50  0000 C CNN
+F 1 "CONN_01X03" V 2424 2745 50  0000 C CNN
 F 2 "Socket_Strips:Socket_Strip_Straight_1x03" H 2300 2750 50  0001 C CNN
 F 3 "" H 2300 2750 50  0000 C CNN
@@
 Text Label 5000 3200 0    60   ~ 0
 RST
+$Comp
+L LD1117S33TR U1
+U 1 1 582742FF
+P 6050 1650
+F 0 "U1" H 6050 2058 50  0000 C CNN
+F 1 "LD1117S33TR" H 6050 1967 50  0000 C CNN
+F 2 "TO_SOT_Packages_THT:TO-220_Neutral123_Vertical" H 6050 1876 50  0000 C CNN
+F 3 "" H 6050 1650 50  0000 C CNN
+	1    6050 1650
+	-1   0    0    -1
+$EndComp
 $EndSCHEMATC
