File: esp8266/esp8266.sch (KiCad schematic (older format))
At the start: 18 parts, among them J1 Screw_Terminal_1x02, J2 Screw_Terminal_1x03, P1 CONN_02X04, P2 CONN_01X03, P3 CONN_01X03, P4 CONN_01X03, P5 CONN_01X03, P6 CONN_01X03, U1 LD1117S33TR

Commit message: add component description to back silk
Parts:
- D1: symbol D -> D-RESCUE-esp8266
- J1: symbol Screw_Terminal_1x02 -> Screw_Terminal_1x02-RESCUE-esp8266
Changed lines of the file:
@@
 EESchema Schematic File Version 2
+LIBS:esp8266-rescue
 LIBS:power
 LIBS:device
@@
 $EndComp
 $Comp
-L D D1
+L D-RESCUE-esp8266 D1
 U 1 1 5823A53F
 P 7050 1600
@@
 $EndComp
 $Comp
-L Screw_Terminal_1x02 J1
+L Screw_Terminal_1x02-RESCUE-esp8266 J1
 U 1 1 5823AAE7
 P 3650 1800

Commit message: add C3
Parts:
- added C3: C_Small, Capacitors_ThroughHole:C_Disc_D3_P2.5, symbol C_Small
- R1, R2, R3: footprint Resistors_THT:Resistor_Horizontal_RM10mm -> Resistors_ThroughHole:Resistor_Horizontal_RM10mm
Connections:
- net +3V3: now also C3.1
- net GND: now also C3.2
Changed lines of the file:
@@
 LIBS:valves
 LIBS:esp8266-cache
-EELAYER 25 0
+EELAYER 26 0
 EELAYER END
 $Descr A4 11693 8268
@@
 F 0 "R3" V 3330 3200 50  0000 C CNN
 F 1 "4.7k" V 3250 3200 50  0000 C CNN
-F 2 "Resistors_THT:Resistor_Horizontal_RM10mm" V 3180 3200 50  0001 C CNN
+F 2 "Resistors_ThroughHole:Resistor_Horizontal_RM10mm" V 3180 3200 50  0001 C CNN
 F 3 "" H 3250 3200 50  0000 C CNN
 	1    3250 3200
@@
 F 0 "R2" V 4930 3150 50  0000 C CNN
 F 1 "2.2k" V 4850 3150 50  0000 C CNN
-F 2 "Resistors_THT:Resistor_Horizontal_RM10mm" V 4780 3150 50  0001 C CNN
+F 2 "Resistors_ThroughHole:Resistor_Horizontal_RM10mm" V 4780 3150 50  0001 C CNN
 F 3 "" H 4850 3150 50  0000 C CNN
 	1    4850 3150
@@
 F 0 "R1" V 4730 3150 50  0000 C CNN
 F 1 "2.2k" V 4650 3150 50  0000 C CNN
-F 2 "Resistors_THT:Resistor_Horizontal_RM10mm" V 4580 3150 50  0001 C CNN
+F 2 "Resistors_ThroughHole:Resistor_Horizontal_RM10mm" V 4580 3150 50  0001 C CNN
 F 3 "" H 4650 3150 50  0000 C CNN
 	1    4650 3150
@@
 Wire Wire Line
 	3850 1900 3950 1900
+$Comp
+L GND #PWR014
+U 1 1 5894FA52
+P 5350 3650
+F 0 "#PWR014" H 5350 3400 50  0001 C CNN
+F 1 "GND" H 5350 3500 50  0000 C CNN
+F 2 "" H 5350 3650 50  0000 C CNN
+F 3 "" H 5350 3650 50  0000 C CNN
+	1    5350 3650
+	1    0    0    -1
+$EndComp
+$Comp
+L C_Small C3
+U 1 1 5894FAF9
+P 5350 3500
+F 0 "C3" H 5442 3546 50  0000 L CNN
+F 1 "C_Small" H 5442 3455 50  0000 L CNN
+F 2 "Capacitors_ThroughHole:C_Disc_D3_P2.5" H 0   0   50  0001 C CNN
+F 3 "" H 0   0   50  0001 C CNN
+	1    5350 3500
+	1    0    0    -1
+$EndComp
+Wire Wire Line
+	5350 3400 5050 3400
+Connection ~ 5050 3400
+Wire Wire Line
+	5350 3600 5350 3650
 $EndSCHEMATC

Commit message: kicad 5
Parts:
- C1, C2: symbol CP -> esp8266-rescue:CP
- C3: symbol C_Small -> esp8266-rescue:C_Small
- D1: symbol D-RESCUE-esp8266 -> esp8266-rescue:D-RESCUE-esp8266
- J1: symbol Screw_Terminal_1x02-RESCUE-esp8266 -> esp8266-rescue:Screw_Terminal_1x02-RESCUE-esp8266
- J2: symbol Screw_Terminal_1x03 -> esp8266-rescue:Screw_Terminal_1x03
- JP1: symbol JUMPER_NO_Small -> esp8266-rescue:JUMPER_NO_Small
- P1: symbol CONN_02X04 -> esp8266-rescue:CONN_02X04
- P2, P3, P4, P5, P6: symbol CONN_01X03 -> esp8266-rescue:CONN_01X03
- PROG1, RESET1: symbol SW_PUSH -> esp8266-rescue:SW_PUSH
- R1, R2, R3: symbol R -> esp8266-rescue:R
- U1: symbol LD1117S33TR -> esp8266-rescue:LD1117S33TR
Connections:
- wire segments 56 -> 72
Changed lines of the file:
@@
-EESchema Schematic File Version 2
-LIBS:esp8266-rescue
-LIBS:power
-LIBS:device
-LIBS:transistors
-LIBS:conn
-LIBS:linear
-LIBS:regul
-LIBS:74xx
-LIBS:cmos4000
-LIBS:adc-dac
-LIBS:memory
-LIBS:xilinx
-LIBS:microcontrollers
-LIBS:dsp
-LIBS:microchip
-LIBS:analog_switches
-LIBS:motorola
-LIBS:texas
-LIBS:intel
-LIBS:audio
-LIBS:interface
-LIBS:digital-audio
-LIBS:philips
-LIBS:display
-LIBS:cypress
-LIBS:siliconi
-LIBS:opto
-LIBS:atmel
-LIBS:contrib
-LIBS:valves
+EESchema Schematic File Version 4
 LIBS:esp8266-cache
 EELAYER 26 0
@@
 $EndDescr
 $Comp
-L CONN_02X04 P1
+L esp8266-rescue:CONN_02X04 P1
 U 1 1 5823A171
 P 5300 3150
@@
 $EndComp
 $Comp
-L CP C2
+L esp8266-rescue:CP C2
 U 1 1 5823A34F
 P 6750 1750
@@
 $EndComp
 $Comp
-L CP C1
+L esp8266-rescue:CP C1
 U 1 1 5823A471
 P 4950 1750
@@
 $EndComp
 $Comp
-L GND #PWR01
+L power:GND #PWR01
 U 1 1 5823A4EB
 P 6050 2000
@@
 $EndComp
 $Comp
-L VCC #PWR02
+L power:VCC #PWR02
 U 1 1 5823A507
 P 7350 1600
@@
 $EndComp
 $Comp
-L +3.3V #PWR03
+L power:+3.3V #PWR03
 U 1 1 5823A523
 P 4800 1600
@@
 $EndComp
 $Comp
-L D-RESCUE-esp8266 D1
+L esp8266-rescue:D-RESCUE-esp8266 D1
 U 1 1 5823A53F
 P 7050 1600
@@
 $EndComp
 $Comp
-L SW_PUSH PROG1
+L esp8266-rescue:SW_PUSH PROG1
 U 1 1 5823A680
 P 6050 3200
@@
 $EndComp
 $Comp
-L GND #PWR04
+L power:GND #PWR04
 U 1 1 5823A808
 P 5700 3000
@@
 $EndComp
 $Comp
-L +3.3V #PWR05
+L power:+3.3V #PWR05
 U 1 1 5823A82F
 P 5050 3450
@@
 $EndComp
 $Comp
-L R R3
+L esp8266-rescue:R R3
 U 1 1 5823A84A
 P 3250 3200
@@
 $EndComp
 $Comp
-L R R2
+L esp8266-rescue:R R2
 U 1 1 5823A89B
 P 4850 3150
@@
 $EndComp
 $Comp
-L R R1
+L esp8266-rescue:R R1
 U 1 1 5823A960
 P 4650 3150
@@
 $EndComp
 $Comp
-L Screw_Terminal_1x02-RESCUE-esp8266 J1
+L esp8266-rescue:Screw_Terminal_1x02-RESCUE-esp8266 J1
 U 1 1 5823AAE7
 P 3650 1800
@@
 $EndComp
 $Comp
-L Screw_Terminal_1x03 J2
+L esp8266-rescue:Screw_Terminal_1x03 J2
 U 1 1 5823AB66
 P 1100 3250
@@
 $EndComp
 $Comp
-L GND #PWR06
+L power:GND #PWR06
 U 1 1 5823ACE3
 P 3950 1900
@@
 $EndComp
 $Comp
-L VCC #PWR07
+L power:VCC #PWR07
 U 1 1 5823AD2F
 P 3950 1700
@@
 $EndComp
 $Comp
-L GND #PWR08
+L power:GND #PWR08
 U 1 1 5823AD6E
 P 2800 3450
@@
 $EndComp
 $Comp
-L +3.3V #PWR09
+L power:+3.3V #PWR09
 U 1 1 5823ADAD
 P 3050 3050
@@
 $EndComp
 $Comp
-L GND #PWR010
+L power:GND #PWR010
 U 1 1 5823C635
 P 3850 2950
@@
 $EndComp
 $Comp
-L SW_PUSH RESET1
+L esp8266-rescue:SW_PUSH RESET1
 U 1 1 5823A79D
 P 4150 2950
@@
 RX
 $Comp
-L GND #PWR011
+L power:GND #PWR011
 U 1 1 5823D32B
 P 6950 2450
@@
 $EndComp
 $Comp
-L CONN_01X03 P2
+L esp8266-rescue:CONN_01X03 P2
 U 1 1 5823AA50
 P 7300 2550
@@
 $EndComp
 $Comp
-L GND #PWR012
+L power:GND #PWR012
 U 1 1 5824925E
 P 6400 3200
@@
 Connection ~ 6750 1600
 Wire Wire Line
-	4800 1600 5650 1600
+	4800 1600 4950 1600
 Connection ~ 4950 1600
 Wire Wire Line
-	3850 1700 4200 1700
-Wire Wire Line
-	1300 3450 2800 3450
-Wire Wire Line
-	1300 3050 3250 3050
+	3850 1700 3950 1700
+Wire Wire Line
+	1300 3450 1400 3450
+Wire Wire Line
+	1300 3050 1600 3050
 Connection ~ 3050 3050
 Wire Wire Line
@@
 	6400 3200 6350 3200
 Wire Wire Line
-	5050 3300 5050 3450
+	5050 3300 5050 3400
 Connection ~ 4850 3300
-Connection ~ 4650 3300
 Wire Wire Line
 	4850 3000 4950 3000
@@
 	4650 3000 4650 2950
 Wire Wire Line
-	4450 2950 5000 2950
+	4450 2950 4650 2950
 Wire Wire Line
 	5000 2950 5000 3200
@@
 Connection ~ 4650 2950
 Wire Wire Line
-	3850 2950 3850 2950
-Wire Wire Line
-	4650 3300 5050 3300
+	4650 3300 4850 3300
 Wire Wire Line
 	5050 2850 5050 3000
@@
 	6050 2000 6050 1900
 Wire Wire Line
-	4950 2000 6750 2000
+	4950 2000 6050 2000
 Wire Wire Line
 	6750 2000 6750 1900
@@
 Connection ~ 6050 2000
 $Comp
-L VDD #PWR013
+L power:VDD #PWR013
 U 1 1 5824AFFA
 P 6750 1450
@@
 	6750 1450 6750 1600
 $Comp
-L CONN_01X03 P3
+L esp8266-rescue:CONN_01X03 P3
 U 1 1 5824B234
 P 1500 2750
@@
 $EndComp
 Wire Wire Line
-	1300 3250 3100 3250
-Wire Wire Line
-	3100 3250 3100 3450
-$Comp
-L CONN_01X03 P4
+	3100 3250 3100 3350
+$Comp
+L esp8266-rescue:CONN_01X03 P4
 U 1 1 5824B795
 P 1900 2750
@@
 $EndComp
 $Comp
-L CONN_01X03 P5
+L esp8266-rescue:CONN_01X03 P5
 U 1 1 5824B805
 P 2300 2750
@@
 $EndComp
 $Comp
-L CONN_01X03 P6
+L esp8266-rescue:CONN_01X03 P6
 U 1 1 5824B867
 P 2700 2750
@@
 	1500 2950 1500 3250
 Wire Wire Line
-	1500 3250 1550 3250
-Connection ~ 1550 3250
-Wire Wire Line
 	1600 2950 1600 3050
 Connection ~ 1600 3050
@@
 Wire Wire Line
 	2600 2950 2600 3450
-Wire Wire Line
-	2600 3450 2550 3450
 Connection ~ 2550 3450
 Wire Wire Line
@@
 Connection ~ 3100 3350
 $Comp
-L JUMPER_NO_Small JP1
+L esp8266-rescue:JUMPER_NO_Small JP1
 U 1 1 5825118E
 P 4300 1350
@@
 RST
 $Comp
-L LD1117S33TR U1
+L esp8266-rescue:LD1117S33TR U1
 U 1 1 582742FF
 P 6050 1650
@@
 	7350 1600 7200 1600
 Wire Wire Line
-	6450 1600 6900 1600
+	6450 1600 6750 1600
 Wire Wire Line
 	3850 1900 3950 1900
 $Comp
-L GND #PWR014
+L power:GND #PWR014
 U 1 1 5894FA52
 P 5350 3650
@@
 $EndComp
 $Comp
-L C_Small C3
+L esp8266-rescue:C_Small C3
 U 1 1 5894FAF9
 P 5350 3500
@@
 Wire Wire Line
 	5350 3600 5350 3650
+Wire Wire Line
+	6750 1600 6900 1600
+Wire Wire Line
+	4950 1600 5650 1600
+Wire Wire Line
+	3050 3050 3250 3050
+Wire Wire Line
+	4850 3300 5050 3300
+Wire Wire Line
+	4650 2950 5000 2950
+Wire Wire Line
+	6050 2000 6750 2000
+Wire Wire Line
+	1400 3450 1800 3450
+Wire Wire Line
+	1600 3050 2000 3050
+Wire Wire Line
+	1800 3450 2200 3450
+Wire Wire Line
+	1900 3250 2300 3250
+Wire Wire Line
+	2000 3050 2400 3050
+Wire Wire Line
+	2300 3250 2700 3250
+Wire Wire Line
+	2400 3050 2800 3050
+Wire Wire Line
+	2700 3250 3100 3250
+Wire Wire Line
+	2800 3050 3050 3050
+Wire Wire Line
+	3100 3350 3100 3450
+Wire Wire Line
+	3950 1700 4200 1700
+Wire Wire Line
+	5050 3400 5050 3450
+Wire Wire Line
+	1300 3250 1900 3250
+Wire Wire Line
+	2200 3450 2800 3450
 $EndSCHEMATC
