File: esp8266/esp8266.kicad_pcb (KiCad board)
At the start: 2 copper layers, 50 x 50 mm, 29 parts, among them J1 Screw_Terminal_1x02, J2 Screw_Terminal_1x03, P1 CONN_02X04, P2 CONN_01X03, P3 CONN_01X03, P4 CONN_01X03, P5 CONN_01X03, P6 CONN_01X03, U1 LD1117S33TR

Commit message: add component description to back silk
Other:
- board text added: "Reference Value C1 10uf C2 100uf P1 ESP8266 R1 R2 2.2k R3 4.7k U1 LD1117S33TR"
Changed lines of the file:
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@@
     (links 51)
     (no_connects 0)
-    (area 134.544999 64.224999 184.695001 114.375001)
+    (area 127.065915 63.0377 190.356943 115.6973)
     (thickness 1.6)
-    (drawings 27)
+    (drawings 28)
     (tracks 206)
     (zones 0)
@@
     (visible_elements FFFFFF7F)
     (pcbplotparams
-      (layerselection 0x010f0_ffffffff)
+      (layerselection 0x00010_7ffffffe)
       (usegerberextensions true)
       (excludeedgelayer true)
@@
     )
   )
+  (gr_text "Reference Value\nC1 10uf\nC2 100uf\nP1 ESP8266\nR1 R2 2.2k\nR3 4.7k\nU1 LD1117S33TR\n" (at 163.83 96.05) (layer B.SilkS)
+    (effects (font (size 1.5 1.5) (thickness 0.3)) (justify mirror))
+  )
   (gr_text + (at 152.4 82.55) (layer F.SilkS)
