File: esp8266/esp8266.kicad_pcb (KiCad board)
At the start: 2 copper layers, 50 x 50 mm, 29 parts, among them J1 Screw_Terminal_1x02, J2 Screw_Terminal_1x03, P1 CONN_02X04, P2 CONN_01X03, P3 CONN_01X03, P4 CONN_01X03, P5 CONN_01X03, P6 CONN_01X03, U1 LD1117S33TR

Commit message: add C3
Parts:
- added C3: C_Small, Capacitors_ThroughHole:C_Disc_D3_P2.5, F.Cu at (173.0, 109.6)
- R1, R2, R3: footprint Resistors_THT:Resistor_Horizontal_RM10mm -> Resistors_ThroughHole:Resistor_Horizontal_RM10mm
Routing:
- net +3V3: track 131.6 -> 133.8 mm
